Commit message: Initial URDF

File: ropy/models/xarco/panda/robots/hand.xacro (robot description, xacro)
@@ -13,5 +13,5 @@
       <visual>
         <geometry>
-          <mesh filename="package://franka_description/meshes/visual/hand.dae"/>
+          <mesh filename="../meshes/visual/hand.dae"/>
         </geometry>
       </visual>
@@ -56,5 +56,5 @@
       <visual>
         <geometry>
-          <mesh filename="package://franka_description/meshes/visual/finger.dae"/>
+          <mesh filename="../meshes/visual/finger.dae"/>
         </geometry>
       </visual>
@@ -64,5 +64,5 @@
         <origin xyz="0 0 0" rpy="0 0 ${pi}"/>
         <geometry>
-          <mesh filename="package://franka_description/meshes/visual/finger.dae"/>
+          <mesh filename="../meshes/visual/finger.dae"/>
         </geometry>
       </visual>

File: ropy/models/xarco/panda/robots/panda_arm.xacro (robot description, xacro)
@@ -14,5 +14,5 @@
       <visual>
         <geometry>
-          <mesh filename="package://${description_pkg}/meshes/visual/link0.dae"/>
+          <mesh filename="../meshes/visual/link0.dae"/>
         </geometry>
       </visual>
@@ -39,5 +39,5 @@
       <visual>
         <geometry>
-          <mesh filename="package://${description_pkg}/meshes/visual/link1.dae"/>
+          <mesh filename="../meshes/visual/link1.dae"/>
         </geometry>
       </visual>
@@ -72,5 +72,5 @@
       <visual>
         <geometry>
-          <mesh filename="package://${description_pkg}/meshes/visual/link2.dae"/>
+          <mesh filename="../meshes/visual/link2.dae"/>
         </geometry>
       </visual>
@@ -105,5 +105,5 @@
       <visual>
         <geometry>
-          <mesh filename="package://${description_pkg}/meshes/visual/link3.dae"/>
+          <mesh filename="../meshes/visual/link3.dae"/>
         </geometry>
       </visual>
@@ -138,5 +138,5 @@
       <visual>
         <geometry>
-          <mesh filename="package://${description_pkg}/meshes/visual/link4.dae"/>
+          <mesh filename="../meshes/visual/link4.dae"/>
         </geometry>
       </visual>
@@ -171,5 +171,5 @@
       <visual>
         <geometry>
-          <mesh filename="package://${description_pkg}/meshes/visual/link5.dae"/>
+          <mesh filename="../meshes/visual/link5.dae"/>
         </geometry>
       </visual>
@@ -222,5 +222,5 @@
       <visual>
         <geometry>
-          <mesh filename="package://${description_pkg}/meshes/visual/link6.dae"/>
+          <mesh filename="../meshes/visual/link6.dae"/>
         </geometry>
       </visual>
@@ -255,5 +255,5 @@
       <visual>
         <geometry>
-          <mesh filename="package://${description_pkg}/meshes/visual/link7.dae"/>
+          <mesh filename="../meshes/visual/link7.dae"/>
         </geometry>
       </visual>
